Commit message: finished nozzle implementation

File: ur_printer_description/urdf/custom_nozzle.xacro (robot description, xacro)
@@ -1,26 +1,56 @@
 <?xml version="1.0"?>
-<robot xmlns:xacro="http://ros.org/wiki/xacro">
-  <xacro:include filename="$(find ur_description)/urdf/ur_macro.xacro"/>
-  <xacro:macro name="custom_nozzle" params="
-    parent
-    *origin
-    ur_type
-    joint_limits_parameters_file
-    kinematics_parameters_file
-    physical_parameters_file
-    visual_parameters_file
-    ">
-    <xacro:ur_robot
-      name="${ur_type}"
-      tf_prefix="${ur_type}_"
-      parent="${parent}"
-      joint_limits_parameters_file="${joint_limits_parameters_file}"
-      kinematics_parameters_file="${kinematics_parameters_file}"
-      physical_parameters_file="${physical_parameters_file}"
-      visual_parameters_file="${visual_parameters_file}"
-      generate_ros2_control_tag="false"
-    >
-      <origin xyz="0 0 0" rpy="0 0 0" />
-    </xacro:ur_robot>
-  </xacro:macro>
-</robot>
+  <robot xmlns:xacro="http://ros.org/wiki/xacro">
+    <xacro:include filename="$(find ur_description)/urdf/ur_macro.xacro"/>
+    <xacro:macro name="custom_nozzle" params="
+      parent
+      *origin
+      ur_type
+      joint_limits_parameters_file
+      kinematics_parameters_file
+      physical_parameters_file
+      visual_parameters_file
+      ">
+      <xacro:ur_robot
+        name="${ur_type}"
+        tf_prefix="${ur_type}_"
+        parent="${parent}"
+        joint_limits_parameters_file="${joint_limits_parameters_file}"
+        kinematics_parameters_file="${kinematics_parameters_file}"
+        physical_parameters_file="${physical_parameters_file}"
+        visual_parameters_file="${visual_parameters_file}"
+        generate_ros2_control_tag="false"
+      >
+        <origin xyz="0 0 0" rpy="0 0 0" />
+      </xacro:ur_robot>
+      <joint name="end_effector_joint" type="fixed">
+        <parent link="ur5e_tool0"/>
+        <child link="end_effector"/>
+        <!-- Adjust position and orientation as needed -->
+        <origin xyz="0.09066 0.17524 -0.0949" rpy="0 0 3.14159"/>
+      </joint>
+      <!-- Define the end effector link with geometries -->
+      <link name="end_effector">
+        <visual>
+          <geometry>
+            <!-- Path to the visual mesh -->
+            <mesh filename="package://ur_printer_description/meshes/EndEffector.stl"/>
+          </geometry>
+          <!-- You can add material/color here if needed -->
+        </visual>
+        <collision>
+          <geometry>
+            <!-- Path to the collision mesh -->
+            <mesh filename="package://ur_printer_description/meshes/EndEffector.stl"/>
+          </geometry>
+        </collision>
+      </link>
+      <!-- Define TCP (Tool Center Point) frame -->
+      <joint name="tcp_joint" type="fixed">
+        <!-- Adjust TCP position as needed, this is the point used for planning -->
+        <origin xyz="0.09087 0.00174 0.09058" rpy="0 0 0"/>
+        <parent link="end_effector"/>
+        <child link="tcp"/>
+      </joint>
+      <link name="tcp"/>
+    </xacro:macro>
+  </robot>

File: ur_printer_description/urdf/test.urdf (robot description, URDF)
Before this commit: robot ur5e_printer, 13 links, 12 joints
Links:
- added link end_effector; collision mesh filename=package://ur_printer_description/meshes/Toolhead2.stl; visual mesh filename=package://ur_printer_description/meshes/Toolhead2.stl
- added link tcp
Joints:
- added joint end_effector_joint: type fixed, parent ur5e_tool0, child end_effector, origin xyz=0 0 0 rpy=0 0 0
- added joint tcp_joint: type fixed, parent end_effector, child tcp, origin xyz=0 0 0.05 rpy=0 0 0
